File: hardware/bricklets.kicad_sch (KiCad schematic)
At the start: 40 parts

Commit message: schematic
Parts:
- C301, C302, C303, C304: value (none) -> 100nF; footprint (none) -> kicad-libraries:C0603F
- CP301, CP302, CP303, CP304, CP305, CP306, CP307, CP308: value (none) -> 220pF; footprint (none) -> kicad-libraries:4X0402
- P301, P302, P303, P304, P305, P306, P307, P308: value (none) -> CON-SENSOR2; footprint (none) -> kicad-libraries:CON-SENSOR2_180
- R301, R302, R303, R304, R305, R306, R307, R308: value (none) -> 100k; footprint (none) -> kicad-libraries:R0402F
- RP301, RP302, RP303, RP304, RP305, RP306, RP307, RP308: value (none) -> 82; footprint (none) -> kicad-libraries:4X0402
- U301, U302, U303, U304: value (none) -> 74AHC244; footprint (none) -> kicad-libraries:TSSOP20
